Commit message: Added Milestone 2 files

File: robot_description/urdf/robot.urdf (robot description, URDF)
Before this commit: robot robot, 7 links, 6 joints
Links:
- link L1: geometry collision cylinder length=0.1 radius=0.08; visual cylinder length=0.1 radius=0.08
- link L2: geometry collision box size=0.1 0.1 0.4; visual box size=0.1 0.1 0.4
- link L3: geometry collision box size=0.4 0.1 0.1; visual box size=0.4 0.1 0.1
- link L4: geometry collision cylinder length=0.1 radius=0.05; visual cylinder length=0.1 radius=0.05
- link L5: geometry collision box size=0.1 0.05 0.05; visual box size=0.1 0.05 0.05
- link L6: geometry collision box size=0.1 0.03 0.03; visual box size=0.1 0.03 0.03
- link base_link: geometry collision box size=0.2 0.2 0.1; visual box size=0.2 0.2 0.1

Commit message: Final updates

File: robot_description/urdf/robot.urdf (robot description, URDF)
Before this commit: robot robot, 7 links, 6 joints
Links:
- added link world
- link L1: mass None -> 1
- link L2: mass None -> 1
- link L3: mass None -> 1
- link L4: mass None -> 1
- link L5: mass None -> 1
- link L6: mass None -> 1
- link base_link: mass None -> 1
Joints:
- added joint virtual_joint: type fixed, parent world, child base_link, origin xyz=0.0 0.0 0.1 rpy=0.0 0.0 0.0
